Commit message: Move camera overhead, drop EE marker boxes, smooth pick-place motion
Camera:
- Relocate the RGBD camera off the gripper to a fixed overhead mount on
  base_link, looking straight down at the workspace, and rename it
  gripper_camera -> overhead_camera everywhere (URDF sensor, gz bridge,
  detector + tuner subscriptions, published optical frame_id, README).
- Delete the unused duplicate gripper_camera xacros under urdf/.
- Add detector.launch.py: runs object_detector and opens rqt_image_view
  already pointed at the annotated detection image.

Remove stray red markers:
- Strip the 1 cm red box visuals from both end-effector frames
  (rh_p12_rn_ee and the UR end_effector_link); keep the frames for
  TF/IK. They rendered at the fingertips and the overhead camera
  detected them as spurious red objects.

Motion (vision_pick_and_place):
- Snap each arm goal to its nearest co-terminal angle before profiling,
  so joints take the short way around instead of spinning ~2 rad the
  long way (the wild transit swings).
- Freeze wrist_3 at the grasp value through the whole carry: a top-down
  grasp is symmetric about vertical, so the hard-coded place poses'
  wrist_3 no longer forces a ~2 rad wrist spin that flung the object.
- Soften the profile (cruise 0.35 rad/s, min move 3.0 s) and log each
  move's max joint travel + planned duration for diagnosis.

Note: keep colon-then-space out of these xacro comments; the sim launch
parses the whole robot_description as YAML and a mapping-key lookalike
breaks it.

File: src/Universal_Robots_ROS2_Description/urdf/ur_macro.xacro (robot description, xacro)
@@ -383,13 +383,8 @@
       <child link="${tf_prefix}end_effector_link"/>
     </joint>
-    <!-- End effector link -->
+    <!-- End effector link (coordinate frame only). Visual removed so the
+         overhead camera does not detect this small red marker box as a
+         stray red object. -->
     <link name="${tf_prefix}end_effector_link">
-      <visual>
-        <origin xyz="0 0 0" rpy="0 0 0"/>
-        <geometry>
-          <box size="0.01 0.01 0.01" />
-        </geometry>
-        <material name="red"/>
-      </visual>
       <inertial>
         <origin xyz="0 0 0" />

File: src/rh_p12_rn_a_description/urdf/rh_p12_rn_a_gripper.xacro (robot description, xacro)
@@ -166,13 +166,13 @@
       <child link="${prefix}rh_p12_rn_ee"/>
     </joint>
-    <!-- Gripper end effector link -->
+    <!-- Gripper end effector link (TCP / grasp frame used by IK).
+         Intentionally has no visual, since it is just a coordinate frame
+         and not a real body. The old 1 cm red box rendered at the
+         fingertips and the overhead camera detected it as a stray red
+         object, so the visual is removed. The frame and its inertial stay
+         intact for TF and kinematics.
+         (Keep this comment free of a colon-then-space, or the sim launch
+         YAML-parse of robot_description will choke.) -->
     <link name="${prefix}rh_p12_rn_ee">
-      <visual>
-        <origin xyz="0 0 0" rpy="0 0 0"/>
-        <geometry>
-          <box size="0.01 0.01 0.01" />
-        </geometry>
-        <material name="red"/>
-      </visual>
       <inertial>
         <origin xyz="0 0 0" />
@@ -183,17 +183,28 @@
       </inertial>
     </link>
-    <gazebo reference="rh_p12_rn_ee">
-      <material>Gazebo/Red</material>
-    </gazebo>
-    <gazebo reference="rh_p12_rn_ee">
-      <material>Gazebo/Red</material>
-    </gazebo>
-    <!-- GRIPPER CAMERA -->
-    <joint type="fixed" name="${prefix}gripper_camera_joint">
-      <origin xyz="0 0.0 0.06" rpy="0 0 0"/>
-      <parent link="${prefix}rh_p12_rn_base"/>
-      <child link="${prefix}gripper_camera_link"/>
-    </joint>
-    <link name="${prefix}gripper_camera_link">
+    <!--
+      OVERHEAD CAMERA (was gripper-mounted).
+      Fixed to base_link (the arm base is bolted to the world, so this is
+      a static, non-moving overhead view) instead of the gripper, so the
+      objects are localized once from a stable top-down view instead of
+      from the moving gripper.
+      Pose is expressed in base_link, using REP-103 axes where
+      X points forward toward the table, Y left, Z up.
+        xyz -> position of the camera above the workspace. TUNE THIS
+               line while watching rqt_image_view until all boxes are
+               centered in frame. x around 0.4 sits it over the boxes,
+               z around 0.8 lifts it well above them.
+        rpy -> "0 1.5708 0" pitches the link's +X axis to point straight
+               down (toward -Z), so the camera looks down at the table.
+      NOTE keep comments free of a colon-followed-by-space here. The sim
+      launch parses the whole robot_description as YAML, and anything that
+      looks like a YAML mapping key inside a comment breaks that parse.
+    -->
+    <joint type="fixed" name="${prefix}overhead_camera_joint">
+      <origin xyz="0.0 0.38 0.8" rpy="0 1.5708 0"/>
+      <parent link="${prefix}base_link"/>
+      <child link="${prefix}overhead_camera_link"/>
+    </joint>
+    <link name="${prefix}overhead_camera_link">
       <inertial>
         <mass value="0.001"/>
@@ -211,10 +222,10 @@
       </visual>
     </link>
-    <joint type="fixed" name="${prefix}gripper_camera_optical_joint">
+    <joint type="fixed" name="${prefix}overhead_camera_optical_joint">
       <origin xyz="0 0 0" rpy="-1.5707 0 -1.5707"/>
-      <parent link="${prefix}gripper_camera_link"/>
-      <child link="${prefix}gripper_camera_optical_link"/>
-    </joint>
-    <link name="${prefix}gripper_camera_optical_link"/>
+      <parent link="${prefix}overhead_camera_link"/>
+      <child link="${prefix}overhead_camera_optical_link"/>
+    </joint>
+    <link name="${prefix}overhead_camera_optical_link"/>
   </xacro:macro>
 </robot>
